File: Schematics/transformer-driven/pga460_transformer.sch (EAGLE design)
At the start: 16 parts, among them IC1 PGA460TPWQ1

Commit message: update report. add in mega shield template.
Parts:
- removed C6: (no value), adafruit:C-USC0805
- removed J1: (no value), SparkFun-Connectors:CONN_05
- removed J2: (no value), SparkFun-Connectors:CONN_02
- added C7: 390pF, adafruit:C-USC0805
- added C8: 0.033uF, adafruit:C-USC0805
- added MURATA: ma59mf14-7n, SparkFun-Connectors:CONN_02
- added R7: 3K, rcl:R-US_M0805
- added R8: 0, adafruit:R-US_M0805
- added T1: B78416A2232A003, SamacSys_Parts:B78416A2232A003
- C1, C3: value (none) -> 0.1uF
- C2: value (none) -> 0.1 uF
- C4: value (none) -> 100uF
- C5: value (none) -> 680pF
- D1: value 1N4004 -> 1N4007; device diode:1N4004 -> casovac:1N4007
- R1: value (none) -> 10
- R2, R3, R4: value (none) -> 10k
- R5: value (none) -> 100
- R6: value (none) -> 2.7k
Connections:
- net N$5 renamed SCLK
- net N$6 renamed TEST
- net RXD renamed RX2
- net TXD renamed TX2
- new net N$10: C7.2, R7.1
- new net N$8: C5.2, MURATA.1, R6.1, R7.2, T1.4
- net GND: now also C4.1, C5.1, C8.2, MURATA.2, R6.2, R8.1, R8.2, T1.6
- net INN: now also C8.1
- net INP: now also C7.1
- net OUTA: now also T1.1
- net OUTB: now also T1.3
- net VPWR: now also C4.2, R5.1, R5.2, T1.2
Other:
- moved on the sheet: C1, C2, C3, C4, C5, R1, R2, R3, R4, R5, R6

Commit message: update layout for transformer-driven
Parts:
- removed R8: 0, adafruit:R-US_M0805
- added 5V/GND: (no value), con-lsta:FE05-2
- added B1: ARDUINO_MEGA_R3FULL, SparkFun-Boards:ARDUINO_MEGA_R3FULL
- added C10, C17: 100uF, adafruit:C-USC0805
- added C11, C18: 680pF, adafruit:C-USC0805
- added C12, C19: 0.1 uF, adafruit:C-USC0805
- added C13, C20: 390pF, adafruit:C-USC0805
- added C14, C21: 0.033uF, adafruit:C-USC0805
- added C15, C16, C6, C9: 0.1uF, adafruit:C-USC0805
- added D2, D3: 1N4007, casovac:1N4007
- added IC2, IC3: PGA460TPWQ1, PGA460TPWQ1:PGA460TPWQ1
- added MCP2515: (no value), con-lsta:FE07-1
- added MURATA1, MURATA2: ma59mf14-7n, SparkFun-Connectors:CONN_02
- added POWER, VIN: (no value), SparkFun-Connectors:CONN_02
- added R10, R11, R12, R18, R19, R20: 10k, adafruit:R-US_R0805
- added R13, R21: 100, adafruit:R-US_R0805
- added R14, R22: 2.7k, adafruit:R-US_R0805
- added R15, R23: 3K, rcl:R-US_M0805
- added R17, R9: 10, adafruit:R-US_R0805
- added T2, T3: B78416A2232A003, SamacSys_Parts:B78416A2232A003
Connections:
- net INN renamed INN_1
- net INP renamed INP_1
- net N$2 renamed IOREG1
- net N$3 renamed AVDD1
- net OUTA renamed OUTA_1
- net OUTB renamed OUTB_1
- removed net N$1: C1.2, IC1.VPWR, R1.2
- new net AVDD2: C12.2, IC2.AVDD
- new net AVDD3: C19.2, IC3.AVDD
- new net CS: B1.53/!CS, MCP2515.3
- new net INN_2: C14.1, IC2.INN
- new net INN_3: C21.1, IC3.INN
- new net INP_2: C13.1, IC2.INP
- new net INP_3: C20.1, IC3.INP
- new net INT: MCP2515.7
- new net IOREG2: C9.2, IC2.IOREG
- new net IOREG3: C16.2, IC3.IOREG
- new net MISO: B1.50/MISO, MCP2515.4
- new net MOSI: B1.51/MOSI, MCP2515.5
- new net N$11: C11.2, MURATA1.1, R14.1, R15.2, T2.4
- new net N$12: C13.2, R15.1
- new net N$16: D3.C, R17.1
- new net N$17: C18.2, MURATA2.1, R22.1, R23.2, T3.4
- new net N$18: C20.2, R23.1
- new net N$9: D2.C, R9.1
- new net OUTA_2: IC2.OUTA, T2.1
- new net OUTA_3: IC3.OUTA, T3.1
- new net OUTB_2: IC2.OUTB, T2.3
- new net OUTB_3: IC3.OUTB, T3.3
- new net RX1: B1.19(RX1), IC1.RXD
- new net RX3: B1.15(RX3), IC3.RXD
- new net SCLK1: IC1.SCLK, R4.2
- new net SCLK2: IC2.SCLK, R12.2
- new net SCLK3: IC3.SCLK, R20.2
- new net TX1: B1.18(TX1), IC1.TXD, R3.2
- new net TX3: B1.14(TX3), IC3.TXD, R19.2
- new net VIN: B1.VIN, C1.2, C15.2, C6.2, D1.A, D2.A, D3.A, IC1.VPWR, IC2.VPWR, IC3.VPWR, POWER.1, R1.2, R13.2, R17.2, R21.2, R5.2, R9.2, VIN.1, VIN.2
- net 5V: now also 5V/GND.1, 5V/GND.3, 5V/GND.5, 5V/GND.7, 5V/GND.9, B1.5V, MCP2515.1, R10.1, R11.1, R18.1, R19.1
- net GND: now also 5V/GND.10, 5V/GND.2, 5V/GND.4, 5V/GND.6, 5V/GND.8, B1.GND, B1.GND@2, C10.1, C11.1, C12.1, C14.2, C15.1, C16.1, C17.1, C18.1, C19.1, C21.2, C6.1, C9.1, IC2.GNDP, IC2.GND_1, IC2.GND_2, IC3.GNDP, IC3.GND_1, IC3.GND_2, MCP2515.2, MURATA1.2, MURATA2.2, POWER.2, R12.1, R14.2, R20.1, R22.2, T2.6, T3.6; no longer R8.1, R8.2
- net RX2: now also B1.17(RX2), IC2.RXD; no longer IC1.RXD
- net SCLK: now also B1.52/SCK, MCP2515.6; no longer IC1.SCLK, R4.2
- net TEST: now also IC2.TEST, IC3.TEST, R10.2, R18.2
- net TX2: now also B1.16(TX2), IC2.TXD, R11.2; no longer IC1.TXD, R3.2
- net VPWR: now also C10.2, C17.2, R13.1, R21.1, T2.2, T3.2; no longer D1.A, R5.2

Commit message: update layout
Connections:
- net N$11 renamed S2+
- net N$17 renamed S3+
- net N$8 renamed S1+
- removed net N$16: D3.C, R17.1
- removed net N$4: D1.C, R1.1
- removed net N$9: D2.C, R9.1
- removed net TEST: IC1.TEST, IC2.TEST, IC3.TEST, R10.2, R18.2, R2.2
- removed net VPWR: C10.2, C17.2, C4.2, R13.1, R21.1, R5.1, T1.2, T2.2, T3.2
- new net S2-: C11.1, C14.2, C5.1, C8.2, MURATA.2, MURATA1.2, R14.2, R6.2, T1.6, T2.6
- new net S3-: C18.1, C21.2, MURATA2.2, R22.2, T3.6
- new net TEST1: IC1.TEST, R2.2
- new net TEST2: IC2.TEST, R10.2
- new net TEST3: IC3.TEST, R18.2
- net GND: no longer C11.1, C14.2, C18.1, C21.2, C5.1, C8.2, MURATA.2, MURATA1.2, MURATA2.2, R14.2, R22.2, R6.2, T1.6, T2.6, T3.6
- net RX1: now also IC1.TXD, R3.2; no longer IC1.RXD
- net RX2: now also IC2.TXD, R11.2; no longer IC2.RXD
- net RX3: now also IC3.TXD, R19.2; no longer IC3.RXD
- net TX1: now also IC1.RXD; no longer IC1.TXD, R3.2
- net TX2: now also IC2.RXD; no longer IC2.TXD, R11.2
- net TX3: now also IC3.RXD; no longer IC3.TXD, R19.2
- net VIN: now also C10.2, C17.2, C4.2, D1.C, D2.C, D3.C, R1.1, R13.1, R17.1, R21.1, R5.1, R9.1, T1.2, T2.2, T3.2

Commit message: update layout
Connections:
- removed net S2-: C11.1, C14.2, C5.1, C8.2, MURATA.2, MURATA1.2, R14.2, R6.2, T1.6, T2.6
- removed net S3-: C18.1, C21.2, MURATA2.2, R22.2, T3.6
- net GND: now also C11.1, C14.2, C18.1, C21.2, C5.1, C8.2, MURATA.2, MURATA1.2, MURATA2.2, R14.2, R22.2, R6.2, T1.6, T2.6, T3.6
Changed lines of the file:
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@@
 <wire x1="320.04" y1="-68.58" x2="322.58" y2="-68.58" width="0.1524" layer="91"/>
+</segment>
+<segment>
+<pinref part="C18" gate="G$1" pin="1"/>
+<wire x1="139.7" y1="-190.5" x2="139.7" y2="-193.04" width="0.1524" layer="91"/>
+<pinref part="R22" gate="G$1" pin="2"/>
+<wire x1="139.7" y1="-193.04" x2="147.32" y2="-193.04" width="0.1524" layer="91"/>
+<wire x1="147.32" y1="-193.04" x2="157.48" y2="-193.04" width="0.1524" layer="91"/>
+<wire x1="157.48" y1="-193.04" x2="157.48" y2="-190.5" width="0.1524" layer="91"/>
+<pinref part="MURATA2" gate="G$1" pin="2"/>
+<wire x1="157.48" y1="-190.5" x2="160.02" y2="-190.5" width="0.1524" layer="91"/>
+<pinref part="T3" gate="G$1" pin="6"/>
+<wire x1="124.46" y1="-187.96" x2="124.46" y2="-193.04" width="0.1524" layer="91"/>
+<wire x1="124.46" y1="-193.04" x2="139.7" y2="-193.04" width="0.1524" layer="91"/>
+<pinref part="C21" gate="G$1" pin="2"/>
+<wire x1="157.48" y1="-193.04" x2="157.48" y2="-210.82" width="0.1524" layer="91"/>
+<wire x1="157.48" y1="-210.82" x2="132.08" y2="-210.82" width="0.1524" layer="91"/>
+<junction x="157.48" y="-193.04"/>
+<junction x="139.7" y="-193.04"/>
+<junction x="147.32" y="-193.04"/>
+<pinref part="SUPPLY6" gate="GND" pin="GND"/>
+<junction x="157.48" y="-210.82"/>
+<label x="157.48" y="-193.04" size="1.778" layer="95"/>
+</segment>
+<segment>
+<pinref part="C5" gate="G$1" pin="1"/>
+<wire x1="76.2" y1="-71.12" x2="76.2" y2="-73.66" width="0.1524" layer="91"/>
+<pinref part="R6" gate="G$1" pin="2"/>
+<wire x1="76.2" y1="-73.66" x2="83.82" y2="-73.66" width="0.1524" layer="91"/>
+<wire x1="83.82" y1="-73.66" x2="93.98" y2="-73.66" width="0.1524" layer="91"/>
+<wire x1="93.98" y1="-73.66" x2="93.98" y2="-71.12" width="0.1524" layer="91"/>
+<pinref part="MURATA" gate="G$1" pin="2"/>
+<wire x1="93.98" y1="-71.12" x2="96.52" y2="-71.12" width="0.1524" layer="91"/>
+<pinref part="T1" gate="G$1" pin="6"/>
+<wire x1="60.96" y1="-68.58" x2="60.96" y2="-73.66" width="0.1524" layer="91"/>
+<wire x1="60.96" y1="-73.66" x2="76.2" y2="-73.66" width="0.1524" layer="91"/>
+<pinref part="C8" gate="G$1" pin="2"/>
+<wire x1="93.98" y1="-73.66" x2="93.98" y2="-91.44" width="0.1524" layer="91"/>
+<wire x1="93.98" y1="-91.44" x2="68.58" y2="-91.44" width="0.1524" layer="91"/>
+<junction x="93.98" y="-73.66"/>
+<junction x="76.2" y="-73.66"/>
+<junction x="83.82" y="-73.66"/>
+<pinref part="SUPPLY5" gate="GND" pin="GND"/>
+<junction x="93.98" y="-91.44"/>
+<label x="93.98" y="-73.66" size="1.778" layer="95"/>
+</segment>
+<segment>
+<pinref part="C11" gate="G$1" pin="1"/>
+<wire x1="213.36" y1="-71.12" x2="213.36" y2="-73.66" width="0.1524" layer="91"/>
+<pinref part="R14" gate="G$1" pin="2"/>
+<wire x1="213.36" y1="-73.66" x2="220.98" y2="-73.66" width="0.1524" layer="91"/>
+<wire x1="220.98" y1="-73.66" x2="231.14" y2="-73.66" width="0.1524" layer="91"/>
+<wire x1="231.14" y1="-73.66" x2="231.14" y2="-71.12" width="0.1524" layer="91"/>
+<pinref part="MURATA1" gate="G$1" pin="2"/>
+<wire x1="231.14" y1="-71.12" x2="233.68" y2="-71.12" width="0.1524" layer="91"/>
+<pinref part="T2" gate="G$1" pin="6"/>
+<wire x1="198.12" y1="-68.58" x2="198.12" y2="-73.66" width="0.1524" layer="91"/>
+<wire x1="198.12" y1="-73.66" x2="213.36" y2="-73.66" width="0.1524" layer="91"/>
+<pinref part="C14" gate="G$1" pin="2"/>
+<wire x1="231.14" y1="-73.66" x2="231.14" y2="-91.44" width="0.1524" layer="91"/>
+<wire x1="231.14" y1="-91.44" x2="205.74" y2="-91.44" width="0.1524" layer="91"/>
+<junction x="231.14" y="-73.66"/>
+<junction x="213.36" y="-73.66"/>
+<junction x="220.98" y="-73.66"/>
+<pinref part="SUPPLY3" gate="GND" pin="GND"/>
+<junction x="231.14" y="-91.44"/>
+<junction x="233.68" y="-71.12"/>
+<label x="231.14" y="-73.66" size="1.778" layer="95"/>
 </segment>
 </net>
@@
 <junction x="220.98" y="-63.5"/>
 <label x="231.14" y="-68.58" size="1.778" layer="95"/>
-<junction x="233.68" y="-68.58"/>
 </segment>
 </net>
@@
 </segment>
 </net>
-<net name="S2-" class="0">
-<segment>
-<pinref part="C5" gate="G$1" pin="1"/>
-<wire x1="76.2" y1="-71.12" x2="76.2" y2="-73.66" width="0.1524" layer="91"/>
-<pinref part="R6" gate="G$1" pin="2"/>
-<wire x1="76.2" y1="-73.66" x2="83.82" y2="-73.66" width="0.1524" layer="91"/>
-<wire x1="83.82" y1="-73.66" x2="93.98" y2="-73.66" width="0.1524" layer="91"/>
-<wire x1="93.98" y1="-73.66" x2="93.98" y2="-71.12" width="0.1524" layer="91"/>
-<pinref part="MURATA" gate="G$1" pin="2"/>
-<wire x1="93.98" y1="-71.12" x2="96.52" y2="-71.12" width="0.1524" layer="91"/>
-<pinref part="T1" gate="G$1" pin="6"/>
-<wire x1="60.96" y1="-68.58" x2="60.96" y2="-73.66" width="0.1524" layer="91"/>
-<wire x1="60.96" y1="-73.66" x2="76.2" y2="-73.66" width="0.1524" layer="91"/>
-<pinref part="C8" gate="G$1" pin="2"/>
-<wire x1="93.98" y1="-73.66" x2="93.98" y2="-91.44" width="0.1524" layer="91"/>
-<wire x1="93.98" y1="-91.44" x2="68.58" y2="-91.44" width="0.1524" layer="91"/>
-<junction x="93.98" y="-73.66"/>
-<junction x="76.2" y="-73.66"/>
-<junction x="83.82" y="-73.66"/>
-<pinref part="SUPPLY5" gate="GND" pin="GND"/>
-<junction x="93.98" y="-91.44"/>
-<label x="93.98" y="-71.12" size="1.778" layer="95"/>
-</segment>
-<segment>
-<pinref part="C11" gate="G$1" pin="1"/>
-<wire x1="213.36" y1="-71.12" x2="213.36" y2="-73.66" width="0.1524" layer="91"/>
-<pinref part="R14" gate="G$1" pin="2"/>
-<wire x1="213.36" y1="-73.66" x2="220.98" y2="-73.66" width="0.1524" layer="91"/>
-<wire x1="220.98" y1="-73.66" x2="231.14" y2="-73.66" width="0.1524" layer="91"/>
-<wire x1="231.14" y1="-73.66" x2="231.14" y2="-71.12" width="0.1524" layer="91"/>
-<pinref part="MURATA1" gate="G$1" pin="2"/>
-<wire x1="231.14" y1="-71.12" x2="233.68" y2="-71.12" width="0.1524" layer="91"/>
-<pinref part="T2" gate="G$1" pin="6"/>
-<wire x1="198.12" y1="-68.58" x2="198.12" y2="-73.66" width="0.1524" layer="91"/>
-<wire x1="198.12" y1="-73.66" x2="213.36" y2="-73.66" width="0.1524" layer="91"/>
-<pinref part="C14" gate="G$1" pin="2"/>
-<wire x1="231.14" y1="-73.66" x2="231.14" y2="-91.44" width="0.1524" layer="91"/>
-<wire x1="231.14" y1="-91.44" x2="205.74" y2="-91.44" width="0.1524" layer="91"/>
-<junction x="231.14" y="-73.66"/>
-<junction x="213.36" y="-73.66"/>
-<junction x="220.98" y="-73.66"/>
-<pinref part="SUPPLY3" gate="GND" pin="GND"/>
-<junction x="231.14" y="-91.44"/>
-<label x="231.14" y="-73.66" size="1.778" layer="95"/>
-<junction x="233.68" y="-71.12"/>
-</segment>
-</net>
-<net name="S3-" class="0">
-<segment>
-<pinref part="C18" gate="G$1" pin="1"/>
-<wire x1="139.7" y1="-190.5" x2="139.7" y2="-193.04" width="0.1524" layer="91"/>
-<pinref part="R22" gate="G$1" pin="2"/>
-<wire x1="139.7" y1="-193.04" x2="147.32" y2="-193.04" width="0.1524" layer="91"/>
-<wire x1="147.32" y1="-193.04" x2="157.48" y2="-193.04" width="0.1524" layer="91"/>
-<wire x1="157.48" y1="-193.04" x2="157.48" y2="-190.5" width="0.1524" layer="91"/>
-<pinref part="MURATA2" gate="G$1" pin="2"/>
-<wire x1="157.48" y1="-190.5" x2="160.02" y2="-190.5" width="0.1524" layer="91"/>
-<pinref part="T3" gate="G$1" pin="6"/>
-<wire x1="124.46" y1="-187.96" x2="124.46" y2="-193.04" width="0.1524" layer="91"/>
-<wire x1="124.46" y1="-193.04" x2="139.7" y2="-193.04" width="0.1524" layer="91"/>
-<pinref part="C21" gate="G$1" pin="2"/>
-<wire x1="157.48" y1="-193.04" x2="157.48" y2="-210.82" width="0.1524" layer="91"/>
-<wire x1="157.48" y1="-210.82" x2="132.08" y2="-210.82" width="0.1524" layer="91"/>
-<junction x="157.48" y="-193.04"/>
-<junction x="139.7" y="-193.04"/>
-<junction x="147.32" y="-193.04"/>
-<pinref part="SUPPLY6" gate="GND" pin="GND"/>
-<junction x="157.48" y="-210.82"/>
-<label x="157.48" y="-193.04" size="1.778" layer="95"/>
-</segment>
-</net>
